File: quadcopter.brd (EAGLE design)
At the start: 128 x 128 mm, 67 parts, among them J1 ISP, J4 SIP-10_TH-254X10, M1 MOTOR_PADS, M2 MOTOR_PADS, M3 MOTOR_PADS, M4 MOTOR_PADS, SW1 PUSHBUTTON_SMD-VERTICAL-1, U1 ATMEGA128RFA1, Y1 16MHz

Commit message: New board fixed de cap and bat_gnd
Parts:
- C1, C3, C5, C7: value 100uF -> 220uF
Connections:
- net BAT_GND: now also MOFSET1.SOURCE, MOFSET2.SOURCE, MOFSET3.SOURCE, MOFSET4.SOURCE
- net GND: no longer MOFSET1.SOURCE, MOFSET2.SOURCE, MOFSET3.SOURCE, MOFSET4.SOURCE
Routing:
- net GND: track 488.0 -> 420.5 mm, vias 15 -> 18
- net BAT_GND: track 48.2 -> 62.3 mm, vias 5 -> 9
